Commit message: feat:changed the sizes to fix the lidar issue

File: model/robot.xacro (robot description, xacro)
@@ -118,10 +118,10 @@
     <visual>
         <geometry>
-            <sphere radius="${r/2}"/>
+            <sphere radius="${r}"/>
         </geometry>
     </visual>
     <collision>
         <geometry>
-            <sphere radius="${r/2}"/>
+            <sphere radius="${r}"/>
         </geometry>
     </collision>
@@ -145,4 +145,10 @@
         </geometry>
   </visual>
+  <collision>
+        <origin xyz="0 0 0" rpy="0 0 0" />
+        <geometry>
+            <cylinder radius="0.1" length="0.1" />
+        </geometry>
+  </collision>
   <inertial>
         <mass value="1e-6"/>
@@ -154,5 +160,5 @@
     <parent link="body_link"/>
     <child link="lidar_link"/>
-    <origin xyz="0 0 ${b+r}" rpy="0 0 0"/>
+    <origin xyz="0 0 ${s1+0.05}" rpy="1.5708 0 0"/>
     <axis xyz="0 1 0" rpy="0 0 0" />
 </joint>

Commit message: feat:fixed the lidar issues and checked points formation working properly

File: model/robot.xacro (robot description, xacro)
@@ -160,5 +160,5 @@
     <parent link="body_link"/>
     <child link="lidar_link"/>
-    <origin xyz="0 0 ${s1+0.05}" rpy="1.5708 0 0"/>
+    <origin xyz="0 0 ${s1+0.05}" rpy="0 0 0"/>
     <axis xyz="0 1 0" rpy="0 0 0" />
 </joint>
